File: hardware/cabinet-locker.sch (KiCad schematic (older format))
At the start: 0 parts

Commit message: Power module
Parts:
- added J1: Debug, Connector_PinHeader_1.27mm:PinHeader_2x03_P1.27mm_Vertical_SMD, symbol Connector_Generic:Conn_02x03_Odd_Even
- added PS?: HLK-PM12, Converter_ACDC:Converter_ACDC_HiLink_HLK-PMxx, symbol Converter_ACDC:HLK-PM12
- added U1: E73-2G4M08S1C, IoT_Home:E73-2G4M08S1C, symbol IoT_Home:E73-2G4M08S1C
Connections:
- new net +12V: PS?.4 (+Vout)
- new net +3V3: J1.1 (Pin_1), U1.19 (VDD), U1.23 (VDDH)
- new net GND: J1.5 (Pin_5), PS?.3 (-Vout), U1.21 (GND), U1.24 (GND), U1.5 (GND)
- new net LINE: PS?.1 (AC/L)
- new net NEUT: PS?.2 (AC/N)
- new net SWDCLK: J1.2 (Pin_2), U1.39 (SWDCLK)
- new net SWDIO: J1.4 (Pin_4), U1.37 (SWDIO)
- new net SWO: J1.6 (Pin_6), U1.36 (P1.00)
- no-connect marks 0 -> 36
Changed lines of the file:
@@
 Comment4 ""
 $EndDescr
+$Comp
+L IoT_Home:E73-2G4M08S1C U1
+U 1 1 5E514202
+P 5300 3800
+F 0 "U1" H 5500 2450 50  0000 C CNN
+F 1 "E73-2G4M08S1C" H 5750 2550 50  0000 C CNN
+F 2 "IoT_Home:E73-2G4M08S1C" H 5300 3700 50  0001 C CNN
+F 3 "http://www.ebyte.com/en/downpdf.aspx?id=445" H 5300 5000 50  0001 C CNN
+	1    5300 3800
+	1    0    0    -1
+$EndComp
+$Comp
+L power:+3.3V #PWR01
+U 1 1 5E5153A0
+P 5250 2450
+F 0 "#PWR01" H 5250 2300 50  0001 C CNN
+F 1 "+3.3V" H 5265 2623 50  0000 C CNN
+F 2 "" H 5250 2450 50  0001 C CNN
+F 3 "" H 5250 2450 50  0001 C CNN
+	1    5250 2450
+	1    0    0    -1
+$EndComp
+$Comp
+L Connector_Generic:Conn_02x03_Odd_Even J1
+U 1 1 5E51628D
+P 7400 4300
+F 0 "J1" H 7450 4617 50  0000 C CNN
+F 1 "Debug" H 7450 4526 50  0000 C CNN
+F 2 "Connector_PinHeader_1.27mm:PinHeader_2x03_P1.27mm_Vertical_SMD" H 7400 4300 50  0001 C CNN
+F 3 "~" H 7400 4300 50  0001 C CNN
+	1    7400 4300
+	1    0    0    -1
+$EndComp
+Text Label 7700 4200 0    50   ~ 0
+SWDCLK
+Text Label 7700 4300 0    50   ~ 0
+SWDIO
+Text Label 7700 4400 0    50   ~ 0
+SWO
+NoConn ~ 7200 4300
+$Comp
+L power:+3.3V #PWR02
+U 1 1 5E51755F
+P 7150 4150
+F 0 "#PWR02" H 7150 4000 50  0001 C CNN
+F 1 "+3.3V" H 7165 4323 50  0000 C CNN
+F 2 "" H 7150 4150 50  0001 C CNN
+F 3 "" H 7150 4150 50  0001 C CNN
+	1    7150 4150
+	1    0    0    -1
+$EndComp
+Wire Wire Line
+	7150 4150 7150 4200
+Wire Wire Line
+	7150 4200 7200 4200
+$Comp
+L power:GND #PWR03
+U 1 1 5E518635
+P 7150 4450
+F 0 "#PWR03" H 7150 4200 50  0001 C CNN
+F 1 "GND" H 7155 4277 50  0000 C CNN
+F 2 "" H 7150 4450 50  0001 C CNN
+F 3 "" H 7150 4450 50  0001 C CNN
+	1    7150 4450
+	1    0    0    -1
+$EndComp
+Wire Wire Line
+	7150 4450 7150 4400
+Wire Wire Line
+	7150 4400 7200 4400
+Text Label 4500 3700 2    50   ~ 0
+SWDCLK
+Text Label 4500 3600 2    50   ~ 0
+SWDIO
+Text Label 4500 4200 2    50   ~ 0
+SWO
+NoConn ~ 4500 3000
+NoConn ~ 4500 2900
+NoConn ~ 4500 4300
+NoConn ~ 4500 4400
+NoConn ~ 4500 4500
+NoConn ~ 4500 4600
+NoConn ~ 4500 4700
+NoConn ~ 4500 4800
+NoConn ~ 4500 4900
+NoConn ~ 6100 4900
+NoConn ~ 6100 4800
+NoConn ~ 6100 4700
+NoConn ~ 6100 4600
+NoConn ~ 6100 4500
+NoConn ~ 6100 4400
+NoConn ~ 6100 4300
+NoConn ~ 6100 4200
+NoConn ~ 6100 4100
+NoConn ~ 6100 4000
+NoConn ~ 6100 3900
+NoConn ~ 6100 3800
+NoConn ~ 6100 3700
+NoConn ~ 6100 3600
+NoConn ~ 6100 3500
+NoConn ~ 6100 3400
+NoConn ~ 6100 3300
+NoConn ~ 6100 3200
+NoConn ~ 6100 3100
+NoConn ~ 6100 3000
+NoConn ~ 6100 2900
+NoConn ~ 6100 2800
+NoConn ~ 6100 2700
+NoConn ~ 5400 2500
+NoConn ~ 5100 2500
+Wire Wire Line
+	5250 2450 5200 2450
+Wire Wire Line
+	5200 2450 5200 2500
+Wire Wire Line
+	5250 2450 5300 2450
+Wire Wire Line
+	5300 2450 5300 2500
+Connection ~ 5250 2450
+$Comp
+L power:GND #PWR04
+U 1 1 5E522538
+P 5300 5100
+F 0 "#PWR04" H 5300 4850 50  0001 C CNN
+F 1 "GND" H 5305 4927 50  0000 C CNN
+F 2 "" H 5300 5100 50  0001 C CNN
+F 3 "" H 5300 5100 50  0001 C CNN
+	1    5300 5100
+	1    0    0    -1
+$EndComp
+NoConn ~ 4500 3800
+$Comp
+L Converter_ACDC:HLK-PM12 PS?
+U 1 1 5E51DD87
+P 2150 1500
+F 0 "PS?" H 2150 1825 50  0000 C CNN
+F 1 "HLK-PM12" H 2150 1734 50  0000 C CNN
+F 2 "Converter_ACDC:Converter_ACDC_HiLink_HLK-PMxx" H 2150 1200 50  0001 C CNN
+F 3 "http://www.hlktech.net/product_detail.php?ProId=56" H 2550 1150 50  0001 C CNN
+	1    2150 1500
+	1    0    0    -1
+$EndComp
+$Comp
+L power:LINE #PWR?
+U 1 1 5E51F2AB
+P 1750 1400
+F 0 "#PWR?" H 1750 1250 50  0001 C CNN
+F 1 "LINE" V 1768 1528 50  0000 L CNN
+F 2 "" H 1750 1400 50  0001 C CNN
+F 3 "" H 1750 1400 50  0001 C CNN
+	1    1750 1400
+	0    -1   -1   0
+$EndComp
+$Comp
+L power:NEUT #PWR?
+U 1 1 5E51F8CA
+P 1750 1600
+F 0 "#PWR?" H 1750 1450 50  0001 C CNN
+F 1 "NEUT" V 1768 1728 50  0000 L CNN
+F 2 "" H 1750 1600 50  0001 C CNN
+F 3 "" H 1750 1600 50  0001 C CNN
+	1    1750 1600
+	0    -1   -1   0
+$EndComp
+$Comp
+L power:+12V #PWR?
+U 1 1 5E51FE85
+P 2600 1350
+F 0 "#PWR?" H 2600 1200 50  0001 C CNN
+F 1 "+12V" H 2615 1523 50  0000 C CNN
+F 2 "" H 2600 1350 50  0001 C CNN
+F 3 "" H 2600 1350 50  0001 C CNN
+	1    2600 1350
+	1    0    0    -1
+$EndComp
+Wire Wire Line
+	2600 1350 2600 1400
+Wire Wire Line
+	2600 1400 2550 1400
+$Comp
+L power:GND #PWR?
+U 1 1 5E5217F3
+P 2600 1650
+F 0 "#PWR?" H 2600 1400 50  0001 C CNN
+F 1 "GND" H 2605 1477 50  0000 C CNN
+F 2 "" H 2600 1650 50  0001 C CNN
+F 3 "" H 2600 1650 50  0001 C CNN
+	1    2600 1650
+	1    0    0    -1
+$EndComp
+Wire Wire Line
+	2600 1650 2600 1600
+Wire Wire Line
+	2600 1600 2550 1600
 $EndSCHEMATC

Commit message: Electromagnet
Parts:
- added D1: 1N4007, Diode_SMD:D_SMA, symbol Diode:1N4007
- added L1: Door Lock, TerminalBlock_RND:TerminalBlock_RND_205-00012_1x02_P5.00mm_Horizontal, symbol Device:Electromagnetic_Actor
- added Q1: AO3400, Package_TO_SOT_SMD:SOT-23, symbol IoT_Home:AO3400
- added R1: 100, symbol Device:R
- added R2: 1M, symbol Device:R
- gave numbers to parts that had none: 1
Connections:
- net +12V: now also D1.1 (K), L1.1 (-)
- net GND: now also Q1.2 (S), R2.2
- new net: D1.2 (A), L1.2 (+), Q1.3 (D)
- new net: Q1.1 (G), R1.1
- new net magnet: R1.2, R2.1
Other:
- moved on the sheet: J1, PS1
Changed lines of the file:
@@
 L Connector_Generic:Conn_02x03_Odd_Even J1
 U 1 1 5E51628D
-P 7400 4300
-F 0 "J1" H 7450 4617 50  0000 C CNN
-F 1 "Debug" H 7450 4526 50  0000 C CNN
-F 2 "Connector_PinHeader_1.27mm:PinHeader_2x03_P1.27mm_Vertical_SMD" H 7400 4300 50  0001 C CNN
-F 3 "~" H 7400 4300 50  0001 C CNN
-	1    7400 4300
-	1    0    0    -1
-$EndComp
-Text Label 7700 4200 0    50   ~ 0
+P 3700 2950
+F 0 "J1" H 3750 3267 50  0000 C CNN
+F 1 "Debug" H 3750 3176 50  0000 C CNN
+F 2 "Connector_PinHeader_1.27mm:PinHeader_2x03_P1.27mm_Vertical_SMD" H 3700 2950 50  0001 C CNN
+F 3 "~" H 3700 2950 50  0001 C CNN
+	1    3700 2950
+	1    0    0    -1
+$EndComp
+Text Label 4000 2850 0    50   ~ 0
 SWDCLK
-Text Label 7700 4300 0    50   ~ 0
+Text Label 4000 2950 0    50   ~ 0
 SWDIO
-Text Label 7700 4400 0    50   ~ 0
+Text Label 4000 3050 0    50   ~ 0
 SWO
-NoConn ~ 7200 4300
-$Comp
-L power:+3.3V #PWR02
+NoConn ~ 3500 2950
+$Comp
+L power:+3.3V #PWR03
 U 1 1 5E51755F
-P 7150 4150
-F 0 "#PWR02" H 7150 4000 50  0001 C CNN
-F 1 "+3.3V" H 7165 4323 50  0000 C CNN
-F 2 "" H 7150 4150 50  0001 C CNN
-F 3 "" H 7150 4150 50  0001 C CNN
-	1    7150 4150
-	1    0    0    -1
-$EndComp
-Wire Wire Line
-	7150 4150 7150 4200
-Wire Wire Line
-	7150 4200 7200 4200
-$Comp
-L power:GND #PWR03
+P 3450 2800
+F 0 "#PWR03" H 3450 2650 50  0001 C CNN
+F 1 "+3.3V" H 3465 2973 50  0000 C CNN
+F 2 "" H 3450 2800 50  0001 C CNN
+F 3 "" H 3450 2800 50  0001 C CNN
+	1    3450 2800
+	1    0    0    -1
+$EndComp
+Wire Wire Line
+	3450 2800 3450 2850
+Wire Wire Line
+	3450 2850 3500 2850
+$Comp
+L power:GND #PWR04
 U 1 1 5E518635
-P 7150 4450
-F 0 "#PWR03" H 7150 4200 50  0001 C CNN
-F 1 "GND" H 7155 4277 50  0000 C CNN
-F 2 "" H 7150 4450 50  0001 C CNN
-F 3 "" H 7150 4450 50  0001 C CNN
-	1    7150 4450
-	1    0    0    -1
-$EndComp
-Wire Wire Line
-	7150 4450 7150 4400
-Wire Wire Line
-	7150 4400 7200 4400
+P 3450 3100
+F 0 "#PWR04" H 3450 2850 50  0001 C CNN
+F 1 "GND" H 3455 2927 50  0000 C CNN
+F 2 "" H 3450 3100 50  0001 C CNN
+F 3 "" H 3450 3100 50  0001 C CNN
+	1    3450 3100
+	1    0    0    -1
+$EndComp
+Wire Wire Line
+	3450 3100 3450 3050
+Wire Wire Line
+	3450 3050 3500 3050
 Text Label 4500 3700 2    50   ~ 0
 SWDCLK
@@
 Connection ~ 5250 2450
 $Comp
-L power:GND #PWR04
+L power:GND #PWR010
 U 1 1 5E522538
 P 5300 5100
-F 0 "#PWR04" H 5300 4850 50  0001 C CNN
+F 0 "#PWR010" H 5300 4850 50  0001 C CNN
 F 1 "GND" H 5305 4927 50  0000 C CNN
 F 2 "" H 5300 5100 50  0001 C CNN
@@
 NoConn ~ 4500 3800
 $Comp
-L Converter_ACDC:HLK-PM12 PS?
+L Converter_ACDC:HLK-PM12 PS1
 U 1 1 5E51DD87
-P 2150 1500
-F 0 "PS?" H 2150 1825 50  0000 C CNN
-F 1 "HLK-PM12" H 2150 1734 50  0000 C CNN
-F 2 "Converter_ACDC:Converter_ACDC_HiLink_HLK-PMxx" H 2150 1200 50  0001 C CNN
-F 3 "http://www.hlktech.net/product_detail.php?ProId=56" H 2550 1150 50  0001 C CNN
-	1    2150 1500
-	1    0    0    -1
-$EndComp
-$Comp
-L power:LINE #PWR?
+P 7400 4650
+F 0 "PS1" H 7400 4975 50  0000 C CNN
+F 1 "HLK-PM12" H 7400 4884 50  0000 C CNN
+F 2 "Converter_ACDC:Converter_ACDC_HiLink_HLK-PMxx" H 7400 4350 50  0001 C CNN
+F 3 "http://www.hlktech.net/product_detail.php?ProId=56" H 7800 4300 50  0001 C CNN
+	1    7400 4650
+	1    0    0    -1
+$EndComp
+$Comp
+L power:LINE #PWR07
 U 1 1 5E51F2AB
-P 1750 1400
-F 0 "#PWR?" H 1750 1250 50  0001 C CNN
-F 1 "LINE" V 1768 1528 50  0000 L CNN
-F 2 "" H 1750 1400 50  0001 C CNN
-F 3 "" H 1750 1400 50  0001 C CNN
-	1    1750 1400
+P 7000 4550
+F 0 "#PWR07" H 7000 4400 50  0001 C CNN
+F 1 "LINE" V 7018 4678 50  0000 L CNN
+F 2 "" H 7000 4550 50  0001 C CNN
+F 3 "" H 7000 4550 50  0001 C CNN
+	1    7000 4550
 	0    -1   -1   0
 $EndComp
 $Comp
-L power:NEUT #PWR?
+L power:NEUT #PWR08
 U 1 1 5E51F8CA
-P 1750 1600
-F 0 "#PWR?" H 1750 1450 50  0001 C CNN
-F 1 "NEUT" V 1768 1728 50  0000 L CNN
-F 2 "" H 1750 1600 50  0001 C CNN
-F 3 "" H 1750 1600 50  0001 C CNN
-	1    1750 1600
+P 7000 4750
+F 0 "#PWR08" H 7000 4600 50  0001 C CNN
+F 1 "NEUT" V 7018 4878 50  0000 L CNN
+F 2 "" H 7000 4750 50  0001 C CNN
+F 3 "" H 7000 4750 50  0001 C CNN
+	1    7000 4750
 	0    -1   -1   0
 $EndComp
 $Comp
-L power:+12V #PWR?
+L power:+12V #PWR06
 U 1 1 5E51FE85
-P 2600 1350
-F 0 "#PWR?" H 2600 1200 50  0001 C CNN
-F 1 "+12V" H 2615 1523 50  0000 C CNN
-F 2 "" H 2600 1350 50  0001 C CNN
-F 3 "" H 2600 1350 50  0001 C CNN
-	1    2600 1350
-	1    0    0    -1
-$EndComp
-Wire Wire Line
-	2600 1350 2600 1400
-Wire Wire Line
-	2600 1400 2550 1400
-$Comp
-L power:GND #PWR?
+P 7850 4500
+F 0 "#PWR06" H 7850 4350 50  0001 C CNN
+F 1 "+12V" H 7865 4673 50  0000 C CNN
+F 2 "" H 7850 4500 50  0001 C CNN
+F 3 "" H 7850 4500 50  0001 C CNN
+	1    7850 4500
+	1    0    0    -1
+$EndComp
+Wire Wire Line
+	7850 4500 7850 4550
+Wire Wire Line
+	7850 4550 7800 4550
+$Comp
+L power:GND #PWR09
 U 1 1 5E5217F3
-P 2600 1650
-F 0 "#PWR?" H 2600 1400 50  0001 C CNN
-F 1 "GND" H 2605 1477 50  0000 C CNN
-F 2 "" H 2600 1650 50  0001 C CNN
-F 3 "" H 2600 1650 50  0001 C CNN
-	1    2600 1650
-	1    0    0    -1
-$EndComp
-Wire Wire Line
-	2600 1650 2600 1600
-Wire Wire Line
-	2600 1600 2550 1600
+P 7850 4800
+F 0 "#PWR09" H 7850 4550 50  0001 C CNN
+F 1 "GND" H 7855 4627 50  0000 C CNN
+F 2 "" H 7850 4800 50  0001 C CNN
+F 3 "" H 7850 4800 50  0001 C CNN
+	1    7850 4800
+	1    0    0    -1
+$EndComp
+Wire Wire Line
+	7850 4800 7850 4750
+Wire Wire Line
+	7850 4750 7800 4750
+$Comp
+L Diode:1N4007 D1
+U 1 1 5E5231FC
+P 7000 2850
+F 0 "D1" V 6954 2929 50  0000 L CNN
+F 1 "1N4007" V 7045 2929 50  0000 L CNN
+F 2 "Diode_SMD:D_SMA" H 7000 2675 50  0001 C CNN
+F 3 "http://www.vishay.com/docs/88503/1n4001.pdf" H 7000 2850 50  0001 C CNN
+	1    7000 2850
+	0    1    1    0
+$EndComp
+$Comp
+L Device:Electromagnetic_Actor L1
+U 1 1 5E524857
+P 7550 2900
+F 0 "L1" H 7680 2996 50  0000 L CNN
+F 1 "Door Lock" H 7680 2905 50  0000 L CNN
+F 2 "TerminalBlock_RND:TerminalBlock_RND_205-00012_1x02_P5.00mm_Horizontal" V 7525 3000 50  0001 C CNN
+F 3 "~" V 7525 3000 50  0001 C CNN
+	1    7550 2900
+	1    0    0    -1
+$EndComp
+Wire Wire Line
+	7000 2700 7550 2700
+Wire Wire Line
+	7000 3000 7550 3000
+$Comp
+L power:+12V #PWR02
+U 1 1 5E526F47
+P 7550 2700
+F 0 "#PWR02" H 7550 2550 50  0001 C CNN
+F 1 "+12V" H 7565 2873 50  0000 C CNN
+F 2 "" H 7550 2700 50  0001 C CNN
+F 3 "" H 7550 2700 50  0001 C CNN
+	1    7550 2700
+	1    0    0    -1
+$EndComp
+Connection ~ 7550 2700
+$Comp
+L IoT_Home:AO3400 Q1
+U 1 1 5E527363
+P 7450 3300
+F 0 "Q1" H 7654 3346 50  0000 L CNN
+F 1 "AO3400" H 7654 3255 50  0000 L CNN
+F 2 "Package_TO_SOT_SMD:SOT-23" H 7650 3225 50  0001 L CIN
+F 3 "http://www.aosmd.com/pdfs/datasheet/ao3400.pdf" H 7450 3300 50  0001 L CNN
+	1    7450 3300
+	1    0    0    -1
+$EndComp
+Text Label 6850 3300 2    50   ~ 0
+magnet
+$Comp
+L Device:R R2
+U 1 1 5E529585
+P 6950 3550
+F 0 "R2" H 7020 3596 50  0000 L CNN
+F 1 "1M" H 7020 3505 50  0000 L CNN
+F 2 "" V 6880 3550 50  0001 C CNN
+F 3 "~" H 6950 3550 50  0001 C CNN
+	1    6950 3550
+	1    0    0    -1
+$EndComp
+$Comp
+L power:GND #PWR05
+U 1 1 5E529B92
+P 7550 3750
+F 0 "#PWR05" H 7550 3500 50  0001 C CNN
+F 1 "GND" H 7555 3577 50  0000 C CNN
+F 2 "" H 7550 3750 50  0001 C CNN
+F 3 "" H 7550 3750 50  0001 C CNN
+	1    7550 3750
+	1    0    0    -1
+$EndComp
+Wire Wire Line
+	7550 3750 7550 3700
+Wire Wire Line
+	6950 3700 7550 3700
+Connection ~ 7550 3700
+Wire Wire Line
+	7550 3700 7550 3500
+Wire Wire Line
+	6950 3400 6950 3300
+Wire Wire Line
+	6950 3300 6850 3300
+$Comp
+L Device:R R1
+U 1 1 5E52FA32
+P 7100 3300
+F 0 "R1" V 6893 3300 50  0000 C CNN
+F 1 "100" V 6984 3300 50  0000 C CNN
+F 2 "" V 7030 3300 50  0001 C CNN
+F 3 "~" H 7100 3300 50  0001 C CNN
+	1    7100 3300
+	0    1    1    0
+$EndComp
+Connection ~ 6950 3300
+Wire Wire Line
+	7550 3100 7550 3000
+Connection ~ 7550 3000
 $EndSCHEMATC
